File: PCB (Eagle)/switch pcb.brd (EAGLE design)
At the start: 27.6 x 25.4 mm, 5 parts

Commit message: Update first release PCB
Parts:
- renumbered U$1 to U$2
Connections:
- net INEFF+: now also U$2.1; no longer U$2.3
- net INJACK+: now also U$2.9; no longer U$2.1
- net INJACK-: now also U$2.10; no longer U$2.4
- net OUTEFF+: now also U$2.3; no longer U$2.7
- net OUTJACK+: now also U$2.7; no longer U$2.9
- net OUTJACK-: now also U$2.4; no longer U$2.10
Routing:
- net INJACK-: track 8.67 -> 23.2 mm
- net OUTJACK+: track 30.7 -> 21.3 mm, vias 0 -> 1
- net INJACK+: track 32.4 -> 38.6 mm
- net INEFF+: track 14.3 -> 17.8 mm
- net OUTJACK-: track 8.67 -> 11.7 mm
- net N$2: track 16.3 -> 14.2 mm
- net OUTEFF+: track 19.5 -> 21.3 mm
- net LED+: track 16.5 -> 15.0 mm, vias 0 -> 1
Other:
- board text added: "InE-"

Commit message: Update switchPCB to version 4423
Corrected footprint for 3PDT switch.
Updated documentation.
Parts:
- turned S2 to 180 degrees
- renumbered S1 to S2
Routing:
- net N$2: track 14.2 -> 27.9 mm
- net OUTEFF+: track 21.3 -> 12.9 mm
- net INJACK+: track 38.6 -> 31.8 mm
- net OUTJACK+: track 21.3 -> 15.0 mm, vias 1 -> 0
Other:
- board text added: "3PDT pcb 4423"
- board text removed: "3PDT pcb 4323"
