File: PCB (Eagle)/SpringReverb.brd (EAGLE design)
At the start: 55 x 45 mm, 36 parts, among them IC2 TL074P, IC3 TLE2426CLP, J1 TB002-500-02BE

Commit message: Update first release PCB
Parts:
- removed IC2: TL074P, linear:DIL14
- removed JP1: (no value), adafruit:1X18
- added C13, C14: 0.1u, rcl:C0603
- added IC1, IC4: TL072P, linear:DIL08
- added JP2: (no value), pinhead:1X04
- added JP4: (no value), pinhead:1X14
- moved R12 24.4 mm to (7.00, 23.5)
- moved R14 20.1 mm to (31.0, 16.0), turned to 0 degrees
- moved R13 19.5 mm to (48.0, 33.5), turned to 90 degrees
- moved R6 18.4 mm to (24.0, 13.0), turned to 180 degrees
- moved C10 17.1 mm to (33.0, 13.5)
- moved R11 15.0 mm to (39.0, 28.5), turned to 180 degrees
- moved R7 14.1 mm to (35.0, 16.0)
- moved C4 14.1 mm to (21.0, 15.5)
- moved C5 12.3 mm to (30.0, 30.5)
- moved R4 12.0 mm to (37.0, 13.0), turned to 90 degrees
- moved C9 8.73 mm to (49.0, 17.5), turned to 270 degrees
- moved R5 8.14 mm to (15.0, 15.5), turned to 0 degrees
- moved C11 7.00 mm to (20.0, 28.0), turned to 0 degrees
- moved H3 7.00 mm to (3.00, 3.00)
- moved H4 7.00 mm to (52.0, 3.00)
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Connections:
- net -12V: now also C14.2, IC1.4, IC4.4; no longer IC2.11
- net 12V: now also C13.1, IC1.8, IC4.8; no longer IC2.4
- net DWELL1: now also JP4.12; no longer JP1.14
- net DWELL2: now also JP4.13; no longer JP1.15
- net EFFIN: now also JP4.1; no longer JP1.1
- net EFFOUT: now also JP4.3; no longer JP1.3
- net GND: now also C13.2, C14.1, IC1.5, IC4.3, IC4.5, JP2.2, JP2.4, JP4.11, JP4.14, JP4.2, JP4.4, JP4.6, JP4.8; no longer IC2.10, IC2.12, IC2.5, JP1.10, JP1.13, JP1.16, JP1.18, JP1.2, JP1.4, JP1.6, JP1.8
- net KILL: now also JP4.7; no longer JP1.9
- net LED: now also JP4.5; no longer JP1.17
- net MIX1: now also JP4.9; no longer JP1.11
- net MIX2: now also JP4.10; no longer JP1.12
- net N$12: now also IC4.2; no longer IC2.9
- net N$13: now also IC4.1; no longer IC2.8
- net N$15: now also IC4.7; no longer IC2.14
- net N$20: now also IC4.6; no longer IC2.13
- net N$3: now also IC1.3; no longer IC2.3
- net N$6: now also IC1.1, IC1.2; no longer IC2.1, IC2.2
- net N$8: now also IC1.6; no longer IC2.6
- net TIN: now also IC1.7, JP2.1; no longer IC2.7, JP1.5
- net TOUT: now also JP2.3; no longer JP1.7
Routing:
- net LED: track 11.0 -> 46.9 mm, vias 0 -> 1
- net N$20: track 10.8 -> 36.3 mm, vias 0 -> 1
- net MIX1: track 36.0 -> 60.5 mm, vias 2 -> 1
- net N$3: track 27.8 -> 6.04 mm
- net N$12: track 27.0 -> 7.16 mm
- net EFFOUT: track 12.0 -> 25.7 mm
- net N$15: track 7.20 -> 20.8 mm
- net DWELL1: track 12.4 -> 20.5 mm, vias 0 -> 1
- net 12V: track 74.9 -> 81.3 mm, vias 1 -> 0
- net MIX2: track 16.7 -> 10.5 mm, vias 1 -> 0
- net KILL: track 33.4 -> 28.3 mm
- net TIN: track 37.6 -> 32.6 mm
- net -12V: track 57.2 -> 62.2 mm
- net EFFIN: track 14.1 -> 18.5 mm
- net DWELL2: track 18.7 -> 15.2 mm
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Other:
- board text added: "DC in"
- board text added: "KILL"
- board text added: "LED"
- board text removed: "24vdc"
- board text removed: "KILL+"
- board text removed: "KILL-"
- board text removed: "LED+"

Commit message: Replaced C6
Replaced C6 (0.1uF) with 22nF for less bass on tank input, therefore less muddy sound
Parts:
- C6: value 0.1u -> 22n
Changed lines of the file:
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@@
 <drawing>
 <settings>
-<setting alwaysvectorfont="yes"/>
+<setting alwaysvectorfont="no"/>
 <setting verticaltext="up"/>
 </settings>
@@
 <attribute name="VALUE" x="16.365" y="28.595" size="1.27" layer="27"/>
 </element>
-<element name="C6" library="rcl" library_urn="urn:adsk.eagle:library:334" package="C0603" package3d_urn="urn:adsk.eagle:package:23616/2" value="0.1u" x="13" y="30.5" smashed="yes" rot="R180">
+<element name="C6" library="rcl" library_urn="urn:adsk.eagle:library:334" package="C0603" package3d_urn="urn:adsk.eagle:package:23616/2" value="22n" x="13" y="30.5" smashed="yes" rot="R180">
 <attribute name="NAME" x="13.635" y="29.865" size="1.27" layer="25" rot="R180"/>
 <attribute name="POPULARITY" value="73" x="13" y="30.5" size="1.778" layer="27" rot="R180" display="off"/>
