File: PCB (Eagle)/SpringReverb.sch (EAGLE design)
At the start: 36 parts, among them IC2 TL074P, IC3 TLE2426CLP, J1 TB002-500-02BE

Commit message: Update first release PCB
Parts:
- removed IC2: TL074P, linear:TL074P
- removed JP1: (no value), adafruit:PINHD-1X18
- added C13, C14: 0.1u, rcl:C-EUC0603
- added IC1, IC4: TL072P, linear:TL072P
- added JP2: (no value), pinhead:PINHD-1X4
- added JP4: (no value), pinhead:PINHD-1X14
Connections:
- net -12V: now also C14.2, IC1P.V-, IC4P.V-; no longer IC2P.V-
- net 12V: now also C13.1, IC1P.V+, IC4P.V+; no longer IC2P.V+
- net DWELL1: now also JP4.12; no longer JP1.14
- net DWELL2: now also JP4.13; no longer JP1.15
- net EFFIN: now also JP4.1; no longer JP1.1
- net EFFOUT: now also JP4.3; no longer JP1.3
- net GND: now also C13.2, C14.1, IC1B.+IN, IC4A.+IN, IC4B.+IN, JP2.2, JP2.4, JP4.11, JP4.14, JP4.2, JP4.4, JP4.6, JP4.8; no longer IC2B.+IN, IC2C.+IN, IC2D.+IN, JP1.10, JP1.13, JP1.16, JP1.18, JP1.2, JP1.4, JP1.6, JP1.8
- net KILL: now also JP4.7; no longer JP1.9
- net LED: now also JP4.5; no longer JP1.17
- net MIX1: now also JP4.9; no longer JP1.11
- net MIX2: now also JP4.10; no longer JP1.12
- net N$12: now also IC4A.-IN; no longer IC2C.-IN
- net N$13: now also IC4A.OUT; no longer IC2C.OUT
- net N$15: now also IC4B.OUT; no longer IC2D.OUT
- net N$20: now also IC4B.-IN; no longer IC2D.-IN
- net N$3: now also IC1A.+IN; no longer IC2A.+IN
- net N$6: now also IC1A.-IN, IC1A.OUT; no longer IC2A.-IN, IC2A.OUT
- net N$8: now also IC1B.-IN; no longer IC2B.-IN
- net TIN: now also IC1B.OUT, JP2.1; no longer IC2B.OUT, JP1.5
- net TOUT: now also JP2.3; no longer JP1.7
Other:
- note added: "Power opamps"
- note removed: "Power TL074"
- moved on the sheet: C11, C12

Commit message: Update with doc
Other:
- note added: "Reverb tank driver -TL072 dual opamp or -NE5532 dual opamp -In and output buffers"
- note removed: "Reverb tank driver -TL074 quad opamp -In and output buffers"
Changed lines of the file:
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@@
 mix</text>
 <text x="15.24" y="-30.48" size="1.778" layer="91">Reverb tank driver
--TL074 quad opamp
+-TL072 dual opamp
+or
+-NE5532 dual opamp
 -In and output buffers</text>
 <text x="-30.48" y="71.12" size="1.778" layer="91">Based on:

Commit message: Replaced C6
Replaced C6 (0.1uF) with 22nF for less bass on tank input, therefore less muddy sound
Parts:
- C6: value 0.1u -> 22n
Changed lines of the file:
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@@
 <part name="C5" library="rcl" library_urn="urn:adsk.eagle:library:334" deviceset="C-EU" device="C1206" package3d_urn="urn:adsk.eagle:package:23618/2" value="0.47u"/>
 <part name="R3" library="rcl" library_urn="urn:adsk.eagle:library:334" deviceset="R-EU_" device="R0603" package3d_urn="urn:adsk.eagle:package:23555/3" value="22k"/>
-<part name="C6" library="rcl" library_urn="urn:adsk.eagle:library:334" deviceset="C-EU" device="C0603" package3d_urn="urn:adsk.eagle:package:23616/2" value="0.1u"/>
+<part name="C6" library="rcl" library_urn="urn:adsk.eagle:library:334" deviceset="C-EU" device="C0603" package3d_urn="urn:adsk.eagle:package:23616/2" value="22n"/>
 <part name="GND2" library="supply1" library_urn="urn:adsk.eagle:library:371" deviceset="GND" device=""/>
 <part name="GND3" library="supply1" library_urn="urn:adsk.eagle:library:371" deviceset="GND" device=""/>
